Commit message: 功能：为 Burger 仿真升级 RGB-D 相机

File: src/turtlebot3_simulations/turtlebot3_gazebo/urdf/turtlebot3_burger_cam.urdf (robot description, URDF)
Before this commit: robot turtlebot3_burger_cam, 10 links, 9 joints
Links:
- added link camera_depth_frame
- added link camera_depth_optical_frame
Joints:
- added joint camera_depth_joint: type fixed, parent camera_link, child camera_depth_frame, origin xyz=0 0 0 rpy=0 0 0
- added joint camera_depth_optical_joint: type fixed, parent camera_depth_frame, child camera_depth_optical_frame, origin xyz=0 0 0 rpy=-1.5707 0 -1.57
- joint camera_joint: origin xyz=0.040 -0.000 0.110 rpy=0 0 0 -> xyz=0.080 0.000 0.250 rpy=0 0 0
- joint camera_rgb_joint: origin xyz=0.003 0.000 0.009 rpy=0 0 0 -> xyz=0 0 0 rpy=0 0 0
